File: Micromouse-Kicad/Micromouse-kicad.kicad_sch (KiCad schematic)
At the start: 97 parts, among them J1 SWD, J2 USB_B_Micro, J3 UARTBTH, J4 Batería, J5 VL6180x, J6 MotorEncodL, J7 MotorEncodR, Q1 BS170, Q2 BS170, Q3 BS170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

Commit message: Fabricado!
Parts:
- J6, J7: footprint Connector_JST:JST_SHL_SM06B-SHLS-TF_1x06-1MP_P1.00mm_Horizontal -> Connector_JST:JST_SH_BM06B-SRSS-TB_1x06-1MP_P1.00mm_Vertical
Connections:
- net GND: now also J4.1 (Pin_1); no longer J4.2 (Pin_2)
- net L_Emitter: now also U1.21 (PA5); no longer U1.22 (PA6)
- net R_Emitter: now also U1.22 (PA6); no longer U1.21 (PA5)
- net VAA: now also J4.2 (Pin_2); no longer J4.1 (Pin_1)
- net DM renamed USB_STM32_D-
- net DP renamed USB_STM32_D+
